File: eagle/BodyCamBoard.brd (EAGLE design)
At the start: 160 x 100 mm, 63 parts, among them IC1 MC33269D-5.0, IC2 TPS77033, IC3 TM4C129XXXPDT, J1 U.FL, Q1 2N3819, Q2 2N3819, U1 RFIDALL, U5 CC3000, X1 USB-A-H, X2 DC21MMX

Commit message: Update main board
Parts:
- removed AE1: ANTENNA22500AT44M0400, SparkFun-RF:ANTENNA-CHIP_2500AT44M0400
- removed C22: 10pF, SparkFun-Capacitors:0603-CAP
- removed C23: DNP, SparkFun-Capacitors:0603-CAP
- removed C24: 2.2pF, SparkFun-Capacitors:0603-CAP
- removed IC2: TPS77033, texas:SOT23-DBV
- removed J1: U.FL, SparkFun-Connectors:U.FL
- removed JP3: Debug, SparkFun-Connectors:1X03
- removed L1: DNP, SparkFun-Passives:0603
- removed L2: 2.2nH, SparkFun-Passives:0603
- removed Q1, Q2: 2N3819, transistor-small-signal:TO92F
- removed SJ2: Mode, SparkFun-Passives:SJ_3_PASTE1&2
- removed TC1: TC2050-IDC-NL, TagConnect:TC2050-IDC-NL
- removed U5: CC3000, SparkFun-RF:QFN-46_CC3000
- removed USBD_N, USBD_P: TEST_POINTSMD_MINI, MAAV_Standard:TEST_SMD_MINI_5019
- added C27, C28: 10uF, SparkFun-Capacitors:0603-CAP
- added JP4: (no value), pinhead:2X03
- added LED2: (no value), SparkFun-LED:LED-0603@1
- added PK4_WAKE, WAKE_SIG: TEST_POINTSMD_MINI, MAAV_Standard:TEST_SMD_MINI_5019
- added R10, R13: 1k, rcl:R0402
- added R11: 1k, resistor:R0603
- added R12: 100, SparkFun-Resistors:0603-RES
- added R14: 10k, resistor:R0603
- added R6: 240, SparkFun-Resistors:0603-RES
- added R7: 390, SparkFun-Resistors:0603-RES
- added R8: 100k, resistor:R0603
- added R9: 180, resistor:R0603
- added U$4, U$5, U$6: IRLML2402TRPBF, MOSFET:SOT-23
- added U$7: 2X5_0.05"_CORTEX_DEBUGTH_KEYED_UNSHROUDED, con-cortex:2X5_0.05"_TH_KEYED_NS
- added U$8: JST_VERTICAL, SparkFun-Connectors:JST-6-SMD-VERT-1.0MM
- added U2: LM1117, SparkFun-PowerIC:SOT223
- C10, C11, C12, C13, C14, C15, C16, C17, C8, C9: device rcl:C0603 -> rcl:C0805
- C21: value 1uF -> 100nf; device SparkFun-Capacitors:0805 -> rcl:C0603
- C6: value 100n -> 0.1uF; device rcl:C0603 -> SparkFun-Capacitors:0603-CAP
- C7: value 100n -> 1uF; device rcl:C0603 -> SparkFun-Capacitors:0603-CAP
- JP2: value (none) -> M09; device pinhead:2X02 -> SparkFun-Connectors:1X09
- LED1: device SparkFun-LED:LED-0603 -> SparkFun-LED:LED-0603@1
- moved RFID_TRIG 415.6 mm to (79.4, 37.9)
- moved SD_CS 376.4 mm to (60.5, 28.4)
- moved SD_CLK 370.9 mm to (55.4, 25.7)
- moved SD_DO 367.9 mm to (55.4, 28.4)
- moved SD_DI 362.6 mm to (60.5, 25.7)
- moved U$3 312.0 mm to (10.9, 33.4), turned to 270 degrees
- moved C26 311.0 mm to (13.5, 34.8), turned to 90 degrees
- moved C25 306.1 mm to (9.33, 36.5)
- moved JP2 292.7 mm to (2.76, 3.27)
- moved D1 291.5 mm to (32.8, 14.2), turned to 270 degrees
- moved X2 271.2 mm to (37.1, 3.56), turned to 180 degrees
- moved C21 269.8 mm to (45.2, 36.1)
- moved C20 256.1 mm to (68.4, 28.3), turned to 180 degrees
- moved R5 252.6 mm to (4.19, 15.5), flipped to the bottom, turned to 270 degrees
- moved C19 252.4 mm to (71.1, 25.4)
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Connections:
- removed net 3.3V: C21.1, U5.P$19, U5.P$23
- removed net JATG_TDO: IC3.97
- removed net N$10: AE1.FEED, C24.1, L1.1
- removed net N$5: C22.1, C24.2, L2.1
- removed net N$6: U5.P$27, U5.P$28
- removed net N$7: U5.P$29, U5.P$30
- removed net N$8: C22.2, C23.1, U5.P$35
- removed net N$9: C23.2, J1.P$3
- removed net NC_4: JP1.9, U$1.7
- removed net WIFI_RX: JP3.2, U5.P$8
- removed net WIFI_TX: JP3.1, U5.P$6
- new net GPS_RXD: IC3.118, U$8.4
- new net GPS_TXD: IC3.119, U$8.3
- new net N$11: R6.1, R7.2, U2.1
- new net N$56: IC3.96, R12.2
- new net PK4_WAKE: IC3.63, PK4_WAKE.P$1, R11.1
- new net RXD: JP4.6, U$1.3
- new net TIVA_LED: IC3.128, LED2.A
- new net TXD: JP4.5, U$1.4
- new net WAKE_SIG: IC3.64, R8.2, U$6.3, WAKE_SIG.P$1
- new net WIFI_EN: IC3.3, JP2.1, R14.2
- net +3V3: now also C28.1, JP2.7, JP4.1, LED1.A, R6.2, R8.1, U$7.1, U2.2, U2.4; no longer IC2.5, JP2.1, LED1.C
- net +5V: now also R12.1, U$8.2; no longer C6.1, IC2.1, IC2.3
- net GND: now also C27.2, C28.2, IC3.80, JP2.9, JP4.2, R10.1, R13.1, R14.1, R7.1, U$4.2, U$5.2, U$6.2, U$7.3, U$7.5, U$7.9, U$8.1, U$8.5; no longer IC2.2, J1.P$1, J1.P$2, JP2.2, JP3.3, L1.2, L2.2, Q1.S, Q2.S, SJ2.3, TC1.3, TC1.5, TC1.9, U5.GND@37, U5.GND@38, U5.GND@39, U5.GND@40, U5.GND@41, U5.GND@42, U5.GND@43, U5.GND@44, U5.GND@45, U5.GND@46, U5.P$1, U5.P$10, U5.P$11, U5.P$16, U5.P$18, U5.P$20, U5.P$21, U5.P$22, U5.P$25, U5.P$26, U5.P$31, U5.P$32, U5.P$33, U5.P$34, U5.P$36, U5.P$9
- net JTAG_TCK: now also U$7.4; no longer TC1.4
- net JTAG_TDI: now also U$7.8; no longer TC1.8
- net JTAG_TDO: now also IC3.97, U$7.6; no longer TC1.6
- net JTAG_TMS: now also U$7.2; no longer TC1.2
- net MIC_TRIG: now also U$1.5; no longer U$1.3
- net N$1: now also LED1.C; no longer LED1.A
- net N$3: now also R9.1; no longer SJ2.2, U5.P$5
- net N$4: now also LED2.C, R9.2; no longer SJ2.1, U5.P$7
- net NC_1: now also JP1.5, U$1.15; no longer JP1.10, U$1.4
- net NC_2: now also JP1.7, U$1.14; no longer JP1.5, U$1.5
- net NC_3: now also JP1.9; no longer JP1.7
- net RESET: now also C21.1, JP4.3, U$7.10; no longer JP2.3, TC1.10
- net RFID_TRIG: now also JP1.10, U$1.7
- net SD_GND: now also U$5.3; no longer Q2.D
- net TEST: now also JP4.4; no longer JP2.4
- net TIVA_WAKE: now also R11.2, U$4.1, U$5.1, U$6.1; no longer IC3.64, Q1.G, Q2.G
- net T_OSC0: now also IC3.88
- net T_OSC1: now also IC3.89
- net USBD_N: now also R10.2; no longer USBD_N.P$1
- net USBD_P: now also R13.2; no longer USBD_P.P$1
- net USB_GND: now also U$4.3; no longer Q1.D
- net VIN: now also C27.1, C6.1, JP2.8, U2.3
- net WIFI_CLK: now also JP2.2; no longer U5.P$17
- net WIFI_CS: now also JP2.4; no longer U5.P$12
- net WIFI_DI: now also JP2.6; no longer U5.P$15
- net WIFI_DO: now also JP2.5; no longer U5.P$13
- net WIFI_INT: now also IC3.126, JP2.3; no longer U5.P$14
Routing:
- net +3V3: track 0.00 -> 341.4 mm, vias 0 -> 11
- net TIVA_WAKE: track 0.00 -> 276.4 mm, vias 0 -> 6
- net +5V: track 0.00 -> 223.1 mm, vias 0 -> 2
- net GND: track 0.00 -> 154.9 mm, vias 0 -> 18
- net VIN: track 0.00 -> 135.4 mm, vias 0 -> 2
- net RESET: track 0.00 -> 117.7 mm, vias 0 -> 2
- net SD_CS: track 0.00 -> 56.7 mm, vias 0 -> 3
- net SD_DO: track 0.00 -> 54.6 mm, vias 0 -> 4
- net SD_DI: track 0.00 -> 49.7 mm, vias 0 -> 4
- net RFID_TRIG: track 0.00 -> 48.3 mm
- net SD_CLK: track 0.00 -> 43.8 mm, vias 0 -> 2
- net NC_3: track 0.00 -> 32.3 mm, vias 0 -> 2
- net WIFI_EN: track 0.00 -> 29.6 mm, vias 0 -> 1
- net SD_GND: track 0.00 -> 27.1 mm
- net NC_2: track 0.00 -> 24.9 mm, vias 0 -> 1
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- added copper zone on layer 1, net GND
- added copper zone on layer 16, net GND
Other:
- board size 160 x 100 mm -> 105.4 x 40.1 mm
- board text added: "Designed by: Jacob Perrin Alec Ten Harmsel Alex LaBerge Yun Han Jiqing Jiang"
- board text added: "EECS 473 Body Cam"
- board text added: "P4_WAKE"
- board text added: "RFID_TRIG"
- board text added: "Version 1.0 10/30/2015"
- board text added: "WAKE_SIG"
