File: eagle/BodyCamBoard.sch (EAGLE design)
At the start: 63 parts, among them IC1 MC33269D-5.0, IC2 TPS77033, IC3 TM4C129XXXPDT, J1 U.FL, Q1 2N3819, Q2 2N3819, U1 RFIDALL, U5 CC3000, X1 USB-A-H, X2 DC21MMX

Commit message: Update main board
Parts:
- removed AE1: ANTENNA22500AT44M0400, SparkFun-RF:ANTENNA22500AT44M0400
- removed C22: 10pF, SparkFun-Capacitors:CAP0603-CAP
- removed C23: DNP, SparkFun-Capacitors:CAP0603-CAP
- removed C24: 2.2pF, SparkFun-Capacitors:CAP0603-CAP
- removed IC2: TPS77033, texas:TPS77033
- removed J1: U.FL, SparkFun-Connectors:U.FL
- removed JP3: Debug, SparkFun-Connectors:M03PTH
- removed L1: DNP, SparkFun-Passives:INDUCTOR0603
- removed L2: 2.2nH, SparkFun-Passives:INDUCTOR0603
- removed Q1, Q2: 2N3819, transistor-small-signal:2N3819
- removed SJ2: Mode, SparkFun-Passives:SOLDERJUMPER_2WAYPASTE1&2
- removed TC1: TC2050-IDC-NL, TagConnect:TC2050-IDC-NL
- removed U5: CC3000, SparkFun-RF:CC3000
- removed USBD_N, USBD_P: TEST_POINTSMD_MINI, MAAV_Standard:TEST_POINTSMD_MINI
- added C27, C28: 10uF, SparkFun-Capacitors:CAP0603-CAP
- added JP4: (no value), pinhead:PINHD-2X3
- added LED2: (no value), SparkFun-LED:LED0603
- added PK4_WAKE, WAKE_SIG: TEST_POINTSMD_MINI, MAAV_Standard:TEST_POINTSMD_MINI
- added R10, R13: 1k, rcl:R-US_R0402
- added R11: 1k, resistor:R-US_R0603
- added R12: 100, SparkFun-Resistors:RESISTOR0603
- added R14: 10k, resistor:R-US_R0603
- added R6: 240, SparkFun-Resistors:RESISTOR0603
- added R7: 390, SparkFun-Resistors:RESISTOR0603
- added R8: 100k, resistor:R-US_R0603
- added R9: 180, resistor:R-US_R0603
- added U$4, U$5, U$6: IRLML2402TRPBF, MOSFET:IRLML2402TRPBF
- added U$7: 2X5_0.05"_CORTEX_DEBUGTH_KEYED_UNSHROUDED, con-cortex:2X5_0.05"_CORTEX_DEBUGTH_KEYED_UNSHROUDED
- added U$8: JST_VERTICAL, SparkFun-Connectors:JST_VERTICAL
- added U2: LM1117, SparkFun-PowerIC:V_REG_LM1117SOT223
- C10, C11, C12, C13, C14, C15, C16, C17, C8, C9: device rcl:C-EUC0603 -> rcl:C-EUC0805
- C21: value 1uF -> 100nf; device SparkFun-Capacitors:CAP0805 -> rcl:C-EUC0603
- C6: value 100n -> 0.1uF; device rcl:C-EUC0603 -> SparkFun-Capacitors:CAP0603-CAP
- C7: value 100n -> 1uF; device rcl:C-EUC0603 -> SparkFun-Capacitors:CAP0603-CAP
- JP2: value (none) -> M09; device pinhead:PINHD-2X2 -> SparkFun-Connectors:M09
Connections:
- removed net 3.3V: C21.1, U5.VBAT_IN, U5.VIO_HOST
- removed net JATG_TDO: IC3.PC3/TDO/SWO
- removed net N$10: AE1.SIGNAL, C24.1, L1.1
- removed net N$5: C22.1, C24.2, L2.1
- removed net N$6: U5.SDA_CC3000, U5.SDA_EEPROM
- removed net N$7: U5.SCL_CC3000, U5.SCL_EEPROM
- removed net N$8: C22.2, C23.1, U5.RF_ANT
- removed net N$9: C23.2, J1.SIGNAL
- removed net NC_4: JP1.9, U$1.7
- removed net WIFI_RX: JP3.2, U5.WL_RS232_RX
- removed net WIFI_TX: JP3.1, U5.WL_RS232_TX
- new net GPS_RXD: IC3.PP0, U$8.4
- new net GPS_TXD: IC3.PP1, U$8.3
- new net N$11: R6.1, R7.2, U2.ADJ
- new net N$56: IC3.PB1, R12.2
- new net PK4_WAKE: IC3.PK4, PK4_WAKE.P$1, R11.1
- new net RXD: JP4.6, U$1.3
- new net TIVA_LED: IC3.PD7, LED2.A
- new net TXD: JP4.5, U$1.4
- new net WAKE_SIG: IC3.!WAKE, R8.2, U$6.D, WAKE_SIG.P$1
- new net WIFI_EN: IC3.PD2, JP2.1, R14.2
- net +3V3: now also C28.1, JP2.7, JP4.1, LED1.A, R6.2, R8.1, U$7.VCC, U2.OUT, U2.OUT@1; no longer IC2.OUT, JP2.1, LED1.C
- net +5V: now also R12.1, U$8.2; no longer C6.1, IC2.!EN, IC2.IN
- net GND: now also C27.2, C28.2, IC3.GND, JP2.9, JP4.2, R10.1, R13.1, R14.1, R7.1, U$4.S, U$5.S, U$6.S, U$7.GND, U$7.GND-DETECT, U$8.1, U$8.5; no longer IC2.GND, J1.GND@0, J1.GND@1, JP2.2, JP3.3, L1.2, L2.2, Q1.S, Q2.S, SJ2.3, TC1.3, TC1.5, TC1.9, U5.EXT_32K, U5.GND@1, U5.GND@10, U5.GND@11, U5.GND@16, U5.GND@18, U5.GND@20, U5.GND@22, U5.GND@25, U5.GND@31, U5.GND@32, U5.GND@33, U5.GND@34, U5.GND@36, U5.GND@37, U5.GND@38, U5.GND@39, U5.GND@40, U5.GND@41, U5.GND@42, U5.GND@43, U5.GND@44, U5.GND@45, U5.GND@46, U5.GND@9, U5.VBAT_SW_EN
- net JTAG_TCK: now also U$7.SWDCLK/TCK; no longer TC1.4
- net JTAG_TDI: now also U$7.NC/TDI; no longer TC1.8
- net JTAG_TDO: now also IC3.PC3/TDO/SWO, U$7.SWO/TDO; no longer TC1.6
- net JTAG_TMS: now also U$7.SWDIO/TMS; no longer TC1.2
- net MIC_TRIG: now also U$1.5; no longer U$1.3
- net N$1: now also LED1.C; no longer LED1.A
- net N$3: now also R9.1; no longer SJ2.2, U5.WL_EN2
- net N$4: now also LED2.C, R9.2; no longer SJ2.1, U5.WL_EN1
- net NC_1: now also JP1.5, U$1.15; no longer JP1.10, U$1.4
- net NC_2: now also JP1.7, U$1.14; no longer JP1.5, U$1.5
- net NC_3: now also JP1.9; no longer JP1.7
- net RESET: now also C21.1, JP4.3, U$7.~RESET; no longer JP2.3, TC1.10
- net RFID_TRIG: now also JP1.10, U$1.7
- net SD_GND: now also U$5.D; no longer Q2.D
- net TEST: now also JP4.4; no longer JP2.4
- net TIVA_WAKE: now also R11.2, U$4.G, U$5.G, U$6.G; no longer IC3.!WAKE, Q1.G, Q2.G
- net T_OSC0: now also IC3.OSC0
- net T_OSC1: now also IC3.OSC1
- net USBD_N: now also R10.2; no longer USBD_N.P$1
- net USBD_P: now also R13.2; no longer USBD_P.P$1
- net USB_GND: now also U$4.D; no longer Q1.D
- net VIN: now also C27.1, C6.1, JP2.8, U2.IN
- net WIFI_CLK: now also JP2.2; no longer U5.SPI_CLK
- net WIFI_CS: now also JP2.4; no longer U5.SPI_CS
- net WIFI_DI: now also JP2.6; no longer U5.SPI_DIN
- net WIFI_DO: now also JP2.5; no longer U5.SPI_DOUT
- net WIFI_INT: now also IC3.PD5, JP2.3; no longer U5.SPI_IRQ
Other:
- note added: "+3V3 power supply"
- note added: "CC3300 WiFi Board plug-in"
- note added: "TIVA Blinky LED"
- note added: "TIVA wake signal circuitry"
- note removed: "+3v3 power supply"
- note removed: "Wifi module & antenna"
- moved on the sheet: C21, C25, C26, C6, C7, D1, LED1, R1, R4, R5, S1
